File: fx502p-sd-pcb-1/fx502p-sd-pcb-1.sch (KiCad schematic (older format))
At the start: 31 parts, among them J1 Conn_01x02_Male, J10 Conn_01x04_Male, J11 Conn_01x04_Male, J3 Conn_01x03_Female, J4 Conn_01x03_Male, J5 Conn_01x10_Male, J6 Conn_01x10_Male, J7 Conn_01x02_Male, P1 Expansion, SW2 Switch_SW_SPST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

Commit message: Removed serial output as it stopped the software serial code from driving the printer once it had initialised (the serial library).
Parts:
- X1: symbol Microtan_exp:XTAL -> fx502p-sd-pcb-1-rescue:XTAL-Microtan_exp
Changed lines of the file:
@@
 	9850 5000 9850 5150
 $Comp
-L Microtan_65_CPU-cache:GND #PWR026
+L fx502p-sd-pcb-1-rescue:GND-Microtan_65_CPU-cache #PWR026
 U 1 1 5FFB06E6
 P 9850 6250
@@
 Connection ~ 5350 3300
 $Comp
-L Microtan_65_CPU-cache:GND #PWR?
+L fx502p-sd-pcb-1-rescue:GND-Microtan_65_CPU-cache #PWR?
 U 1 1 5FFC10FA
 P 4950 7550
@@
 	4000 2750 4000 2350
 $Comp
-L Microtan_exp:XTAL X?
+L fx502p-sd-pcb-1-rescue:XTAL-Microtan_exp X?
 U 1 1 60007C71
 P 5050 1950
@@
 $EndComp
 $Comp
-L Microtan_65_CPU-cache:GND #PWR?
+L fx502p-sd-pcb-1-rescue:GND-Microtan_65_CPU-cache #PWR?
 U 1 1 60007C91
 P 5050 2750
@@
 $EndComp
 $Comp
-L Microtan_65_CPU-cache:GND #PWR?
+L fx502p-sd-pcb-1-rescue:GND-Microtan_65_CPU-cache #PWR?
 U 1 1 60007CA4
 P 3000 1900
@@
 $EndComp
 $Comp
-L Microtan_65_CPU-cache:GND #PWR?
+L fx502p-sd-pcb-1-rescue:GND-Microtan_65_CPU-cache #PWR?
 U 1 1 60007CAA
 P 4500 1450
@@
 CALC_GND
 $Comp
-L Microtan_65_CPU-cache:GND #PWR02
+L fx502p-sd-pcb-1-rescue:GND-Microtan_65_CPU-cache #PWR02
 U 1 1 6003805B
 P 1350 7200
@@
 $EndComp
 $Comp
-L Microtan_65_CPU-cache:GND #PWR03
+L fx502p-sd-pcb-1-rescue:GND-Microtan_65_CPU-cache #PWR03
 U 1 1 60048E05
 P 8050 2950
@@
 $EndComp
 $Comp
-L Microtan_65_CPU-cache:GND #PWR04
+L fx502p-sd-pcb-1-rescue:GND-Microtan_65_CPU-cache #PWR04
 U 1 1 6004E771
 P 2350 2400
@@
 CALC_OP
 $Comp
-L Microtan_65_CPU-cache:GND #PWR06
+L fx502p-sd-pcb-1-rescue:GND-Microtan_65_CPU-cache #PWR06
 U 1 1 6006A9F7
 P 950 4300
@@
 	4450 6900 3050 6900
 $Comp
-L Microtan_65_CPU-cache:GND #PWR08
+L fx502p-sd-pcb-1-rescue:GND-Microtan_65_CPU-cache #PWR08
 U 1 1 60085A8E
 P 3200 7150
@@
 	4450 6100 2550 6100
 $Comp
-L Microtan_65_CPU-cache:GND #PWR05
+L fx502p-sd-pcb-1-rescue:GND-Microtan_65_CPU-cache #PWR05
 U 1 1 600A841C
 P 2700 6350
@@
 $EndComp
 $Comp
-L Microtan_65_CPU-cache:GND #PWR021
+L fx502p-sd-pcb-1-rescue:GND-Microtan_65_CPU-cache #PWR021
 U 1 1 600EAC67
 P 8550 1650
@@
 	8550 1250 9050 1250
 $Comp
-L Microtan_65_CPU-cache:GND #PWR023
+L fx502p-sd-pcb-1-rescue:GND-Microtan_65_CPU-cache #PWR023
 U 1 1 600EE7BA
 P 8550 2600
@@
 Option to power \ncalculator from \nUSB (FX502P only).\nRemove batteries.
 $Comp
-L Microtan_65_CPU-cache:GND #PWR?
+L fx502p-sd-pcb-1-rescue:GND-Microtan_65_CPU-cache #PWR?
 U 1 1 601CED60
 P 5700 2750
@@
 $EndComp
 $Comp
-L Microtan_65_CPU-cache:GND #PWR0101
+L fx502p-sd-pcb-1-rescue:GND-Microtan_65_CPU-cache #PWR0101
 U 1 1 602953AC
 P 7200 5000
@@
 $EndComp
 $Comp
-L Microtan_65_CPU-cache:GND #PWR0102
+L fx502p-sd-pcb-1-rescue:GND-Microtan_65_CPU-cache #PWR0102
 U 1 1 6029CA74
 P 7400 5000
@@
 $EndComp
 $Comp
-L Microtan_65_CPU-cache:GND #PWR0103
+L fx502p-sd-pcb-1-rescue:GND-Microtan_65_CPU-cache #PWR0103
 U 1 1 602A3D07
 P 7600 5000
