File: fx502p-sd-pcb-1/stm_support.sch (KiCad schematic (older format))
At the start: 29 parts, among them J6 Conn_01x05, J7 Conn_01x04, J8 Conn_02x03_Odd_Even, SW1 Switch_SW_SPST, U2 AMS1117-3.3, X2 8MHz

Commit message: Removed serial output as it stopped the software serial code from driving the printer once it had initialised (the serial library).
Parts:
- X2: symbol Microtan_exp:XTAL -> fx502p-sd-pcb-1-rescue:XTAL-Microtan_exp
Changed lines of the file:
@@
 $EndDescr
 $Comp
-L Microtan_65_CPU-cache:GND #PWR?
+L fx502p-sd-pcb-1-rescue:GND-Microtan_65_CPU-cache #PWR?
 U 1 1 5FE7F06A
 P 2050 2650
@@
 AR Path="/5F7FB2B8/5FE7F06A" Ref="#PWR0111"  Part="1"
 AR Path="/5FFAC35B/5FE7F06A" Ref="#PWR030"  Part="1"
+AR Path="/5FE7F06A" Ref="#PWR030"  Part="1"
 F 0 "#PWR030" H 2050 2650 30  0001 C CNN
 F 1 "GND" H 2050 2580 30  0001 C CNN
@@
 $EndComp
 $Comp
-L Microtan_65_CPU-cache:GND #PWR?
+L fx502p-sd-pcb-1-rescue:GND-Microtan_65_CPU-cache #PWR?
 U 1 1 5FE7F09D
 P 4100 1800
@@
 AR Path="/5F7FB2B8/5FE7F09D" Ref="#PWR0112"  Part="1"
 AR Path="/5FFAC35B/5FE7F09D" Ref="#PWR034"  Part="1"
+AR Path="/5FE7F09D" Ref="#PWR034"  Part="1"
 F 0 "#PWR034" H 4100 1800 30  0001 C CNN
 F 1 "GND" H 4100 1730 30  0001 C CNN
@@
 $EndComp
 $Comp
-L Microtan_65_CPU-cache:GND #PWR?
+L fx502p-sd-pcb-1-rescue:GND-Microtan_65_CPU-cache #PWR?
 U 1 1 5FE90D0A
 P 2050 4250
@@
 	6650 1150 6900 1150
 $Comp
-L Microtan_65_CPU-cache:GND #PWR?
+L fx502p-sd-pcb-1-rescue:GND-Microtan_65_CPU-cache #PWR?
 U 1 1 5FED051A
 P 6900 1450
@@
 	7650 2050 8100 2050
 $Comp
-L Microtan_65_CPU-cache:GND #PWR?
+L fx502p-sd-pcb-1-rescue:GND-Microtan_65_CPU-cache #PWR?
 U 1 1 5F95AD5D
 P 6900 2350
@@
 	7700 2900 8150 2900
 $Comp
-L Microtan_65_CPU-cache:GND #PWR?
+L fx502p-sd-pcb-1-rescue:GND-Microtan_65_CPU-cache #PWR?
 U 1 1 5F95FC14
 P 6950 3200
@@
 $EndComp
 $Comp
-L Microtan_65_CPU-cache:GND #PWR?
+L fx502p-sd-pcb-1-rescue:GND-Microtan_65_CPU-cache #PWR?
 U 1 1 6001C4CA
 P 4950 4850
@@
 NRST
 $Comp
-L Microtan_exp:XTAL X?
+L fx502p-sd-pcb-1-rescue:XTAL-Microtan_exp X?
 U 1 1 6001C4E2
 P 4550 5900
@@
 $EndComp
 $Comp
-L Microtan_65_CPU-cache:GND #PWR?
+L fx502p-sd-pcb-1-rescue:GND-Microtan_65_CPU-cache #PWR?
 U 1 1 6001C4F8
 P 3900 6700
@@
 Connection ~ 4950 5600
 $Comp
-L Microtan_65_CPU-cache:GND #PWR?
+L fx502p-sd-pcb-1-rescue:GND-Microtan_65_CPU-cache #PWR?
 U 1 1 6001C513
 P 4550 6700
