File: fx502p-minimal-sd/_autosave-fx502p-minimal-sd.sch (KiCad schematic (older format))
At the start: 20 parts, among them J1 Conn_01x02_Male, J2 Conn_01x02_Male, J3 Conn_01x03_Female, J4 Conn_01x04_Male, J5 Conn_01x04_Male, J6 Conn_01x03_Female, J7 Conn_01x10_Female, P1 Expansion, U1 STM32F103RGTx

Commit message: Update
Parts:
- A1: symbol Charleslabs_Parts:SD_Card_Module_catalex -> fx502p-minimal-sd-rescue:SD_Card_Module_catalex-Charleslabs_Parts
- J1, J2: symbol Connector:Conn_01x02_Male -> fx502p-minimal-sd-rescue:Conn_01x02_Male-Connector
- J3, J6: symbol Connector:Conn_01x03_Female -> fx502p-minimal-sd-rescue:Conn_01x03_Female-Connector
- J4, J5: symbol Connector:Conn_01x04_Male -> fx502p-minimal-sd-rescue:Conn_01x04_Male-Connector
- J7: symbol Connector:Conn_01x10_Female -> fx502p-minimal-sd-rescue:Conn_01x10_Female-Connector
- P1: symbol fx502p:Expansion -> fx502p-minimal-sd-rescue:Expansion-fx502p
- U1: symbol MCU_ST_STM32F1:STM32F103RGTx -> fx502p-minimal-sd-rescue:STM32F103RGTx-MCU_ST_STM32F1
